Commit message: Thruster plugin added to xacro

File: src/rov_description/src/urdf/assembly.xacro (robot description, xacro)
@@ -2,4 +2,3 @@
 <robot name = "ROV" xmlns:xacro="http://ros.org/wiki/xacro">
   <xacro:include filename="core_rov.xacro" />
-  <xacro:include filename="tools/camera.xacro" />
-  <xacro:include filename="tools/gripper.xacro" />
+  <xacro:include filename="tools/thrusters.xacro" />

File: src/rov_description/src/urdf/core_rov.xacro (robot description, xacro)
@@ -22,5 +22,5 @@
     </collision>
   </link>
-  <link name="horizontal_thruster2_1">
+  <link name="horizontal_thruster2">
     <inertial>
       <origin xyz="0.009999999999999898 -0.04000000000000006 -0.04550000000000001" rpy="0 0 0"/>
@@ -31,5 +31,5 @@
       <origin xyz="-0.175 -0.215 -0.21" rpy="0 0 0"/>
       <geometry>
-        <mesh filename="file://$(find ROV_description)/meshes/horizontal_thruster2_1.stl" scale="0.001 0.001 0.001"/>
+        <mesh filename="file://$(find ROV_description)/meshes/horizontal_thruster2.stl" scale="0.001 0.001 0.001"/>
       </geometry>
       <material name="silver"/>
@@ -38,9 +38,9 @@
       <origin xyz="-0.175 -0.215 -0.21" rpy="0 0 0"/>
       <geometry>
-        <mesh filename="file://$(find ROV_description)/meshes/horizontal_thruster2_1.stl" scale="0.001 0.001 0.001"/>
-      </geometry>
-    </collision>
-  </link>
-  <link name="horizontal_thruster4_1">
+        <mesh filename="file://$(find ROV_description)/meshes/horizontal_thruster2.stl" scale="0.001 0.001 0.001"/>
+      </geometry>
+    </collision>
+  </link>
+  <link name="horizontal_thruster4">
     <inertial>
       <origin xyz="1.3877787807814457e-16 0.017000000000000015 -0.04550000000000001" rpy="0 0 0"/>
@@ -51,5 +51,5 @@
       <origin xyz="0.1875 -0.1573 -0.21" rpy="0 0 0"/>
       <geometry>
-        <mesh filename="file://$(find ROV_description)/meshes/horizontal_thruster4_1.stl" scale="0.001 0.001 0.001"/>
+        <mesh filename="file://$(find ROV_description)/meshes/horizontal_thruster4.stl" scale="0.001 0.001 0.001"/>
       </geometry>
       <material name="silver"/>
@@ -58,9 +58,9 @@
       <origin xyz="0.1875 -0.1573 -0.21" rpy="0 0 0"/>
       <geometry>
-        <mesh filename="file://$(find ROV_description)/meshes/horizontal_thruster4_1.stl" scale="0.001 0.001 0.001"/>
-      </geometry>
-    </collision>
-  </link>
-  <link name="vertical_thruster2__1__1">
+        <mesh filename="file://$(find ROV_description)/meshes/horizontal_thruster4.stl" scale="0.001 0.001 0.001"/>
+      </geometry>
+    </collision>
+  </link>
+  <link name="vertical_thruster2">
     <inertial>
       <origin xyz="0.04550000000000004 -0.21499999999999997 -0.009999999999999953" rpy="0 0 0"/>
@@ -71,5 +71,5 @@
       <origin xyz="-0.2 -0.215 -0.235" rpy="0 0 0"/>
       <geometry>
-        <mesh filename="file://$(find ROV_description)/meshes/vertical_thruster2__1__1.stl" scale="0.001 0.001 0.001"/>
+        <mesh filename="file://$(find ROV_description)/meshes/vertical_thruster2.stl" scale="0.001 0.001 0.001"/>
       </geometry>
       <material name="silver"/>
@@ -78,5 +78,5 @@
       <origin xyz="-0.2 -0.215 -0.235" rpy="0 0 0"/>
       <geometry>
-        <mesh filename="file://$(find ROV_description)/meshes/vertical_thruster2__1__1.stl" scale="0.001 0.001 0.001"/>
+        <mesh filename="file://$(find ROV_description)/meshes/vertical_thruster2.stl" scale="0.001 0.001 0.001"/>
       </geometry>
     </collision>
